File: swr_meter.kicad_pcb (KiCad board)
At the start: 4 copper layers, 65 x 70 mm, 68 parts, among them J1 Conn_01x02, J2 Conn_01x02, J3 Conn_01x02_Socket, J4 IDC10, J5 Encoder, U1 AD8307ARZ, U2 AD8307ARZ, U201 TSR1-2450E, U3 ISL60002DIH326Z-TK, U4 AD7991YRJZ-0RL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

Commit message: minor changes, silk cleaning, new ibom
Parts:
- added REF**: OSHW-Logo_5.7x6mm_SilkScreen, Symbol:OSHW-Logo_5.7x6mm_SilkScreen, F.Cu at (122.6, 81.8)
- added REF**: KiCad-Logo2_5mm_SilkScreen, Symbol:KiCad-Logo2_5mm_SilkScreen, F.Cu at (121.0, 63.2)
- U201: moved to F.Cu
- moved C28 6.71 mm to (157.4, 56.8), turned to 0 degrees
- moved C29 5.92 mm to (135.1, 57.0), turned to 0 degrees
- moved C15 4.37 mm to (167.8, 84.6)
- moved C25 4.37 mm to (165.8, 84.6)
- moved C17 4.35 mm to (169.8, 84.6)
- moved J3 3.60 mm to (174.2, 69.0)
- moved U201 1.65 mm to (173.5, 90.7), turned to -90 degrees
- moved C24 1.50 mm to (174.6, 83.0)
Routing:
- net +5V: track 146.6 -> 149.4 mm
- net Net-(J3-Pin_2): track 18.8 -> 20.8 mm
- net GND: vias 228 -> 227
Other:
- board text added: "8-30Vcc"
- board text added: "Encoder"
- board text added: "More info : https://groups.io/g/RadioStuff https://sites.google.com/view/pd0lew/projects/power-and-swr-meter"
- board text added: "Power/SWR Meter PD0LEW"
