File: swr_meter.kicad_sch (KiCad schematic)
At the start: 68 parts, among them J1 Conn_01x02, J2 Conn_01x02, J3 Conn_01x02_Socket, J4 IDC10, J5 Encoder, U1 AD8307ARZ, U2 AD8307ARZ, U201 TSR1-2450E, U3 ISL60002DIH326Z-TK, U4 AD7991YRJZ-0RL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

Commit message: minor changes, silk cleaning, new ibom
Parts:
- renumbered U201 to U6
Changed lines of the file:
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@@
 		(in_pos_files yes)
 		(dnp no)
-		(property "Reference" "U201"
+		(property "Reference" "U6"
 			(at 212.09 11.43 0)
 			(show_name no)
@@
 			(project "swr_meter"
 				(path "/50ae8079-e6ac-4772-9784-7ae19d73aff9"
-					(reference "U201")
+					(reference "U6")
 					(unit 1)
 				)
