File: swr_meter.kicad_sch (KiCad schematic)
At the start: 68 parts, among them J1 Conn_01x02, J2 Conn_01x02, J3 Conn_01x02_Socket, J4 IDC10, J5 Encoder, U1 AD8307ARZ, U2 AD8307ARZ, U3 ISL60002DIH326Z-TK, U4 AD7991YRJZ-0RL, U5 Teensy4.0, U6 TSR1-2450E, U7 PE4259-63, U8 PE4259-63, X1 SMA, X2 U.FL, X3 U.FL, X4 SMA

Commit message: Sorry Johan, typo fixed now
Parts:
- U6: value TSR1-2450E -> TSRN 1-2450E
Other:
- note added: "J.G. Holstein PD0LEW"
- note removed: "J.G. Hostein PD0LEW"
Changed lines of the file:
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@@
 		)
 	)
-	(text "J.G. Hostein\nPD0LEW"
+	(text "J.G. Holstein\nPD0LEW"
 		(exclude_from_sim no)
 		(at 219.71 173.99 0)
@@
 			)
 		)
-		(property "Value" "TSR1-2450E"
+		(property "Value" "TSRN 1-2450E"
 			(at 212.09 13.97 0)
 			(show_name no)
